File: Project/EHM.brd (EAGLE design)
At the start: 78 x 60 mm, 111 parts, among them J1 282834-2, J2 282834-2, J3 282834-2, J4 282834-2, J5 S2B-PH-SM4-TB(LF)(SN), J6 S6B-PH-SM4-TB(LF)(SN), Q1 BC557B, Q2 BC547B, U1 MAX9934TAUA, U2 BQ25570RGRR, U3 TSU111ICT, U4 MAX9934TAUA, U5 TSU111ICT, U6 TSU111ICT

Commit message: Update project to v1.3
Parts:
- added J7: S2B-PH-SM4-TB(LF)(SN), S2B-PH-SM4-TB_LF__SN_:JST_S2B-PH-SM4-TB(LF)(SN)
- C1: value DNP -> 0.01uF; device rcl:C1210 -> rcl:C0805
- C10: value (none) -> 0.1uF
- C11: value 0.01uF -> DNP
- C12: value 4.7uF -> 0.1uF
- C13, C9: value 0.1uF -> 4.7uF
- C14: value DNP -> 0.1uF
- C15: value 4.7uF -> DNP
- C17: value 0.1uF -> DNP
- C2, C3: value 0.01uF -> DNP; device rcl:C0805 -> rcl:C1210
- C21: value DNP -> 0.1uF; device rcl:C1812 -> rcl:C0805
- C22: device rcl:C0805 -> rcl:C1812
- C23: device rcl:C0805 -> rcl:C0603
- C24, C25: value (none) -> 0.1uF; device rcl:C0805 -> rcl:C0603
- C4: value 22uF -> 0.01uF
- C5: value 4.7uF -> 0.01uF
- C6: value 0.1uF -> 22uF
- C7: value DNP -> 4.7uF
- C8: value DNP -> 0.1uF; device rcl:C1210 -> rcl:C0805
- J5: value S2B-PH-SM4-TB(LF)(SN) -> 282834-2; device S2B-PH-SM4-TB_LF__SN_:JST_S2B-PH-SM4-TB(LF)(SN) -> 282834-2:CONN_282834-2
- R1, R10, R12, R13, R5, R9: value DNP -> (none)
- R11, R3: value DNP -> (none); device rcl:R0603 -> Y14870RXX000B9R:Y14870RXX000B9R
- R15, R16, R17, R18, R19, R22, R23: value (none) -> DNP
- R4: device Y14870RXX000B9R:Y14870RXX000B9R -> rcl:R0603
- R8: value (none) -> DNP; device Y14870RXX000B9R:Y14870RXX000B9R -> rcl:R0603
- SJ1, SJ3, SJ8: device jumper:SJ_2 -> jumper:SJ
- SJ13, SJ14, SJ17: device jumper:SJ -> jumper:SJ_2
- TP18: value TPPAD1-13Y -> TPPAD1-13; device testpad:P1-13Y -> testpad:P1-13
- TP23: value TPPAD1-13Y -> TPB1,27; device testpad:P1-13Y -> testpad:B1,27
- U1: value MAX9934TAUA -> BQ25570RGRR; device MAX9934TAUA:21-0036K -> BQ25570RGRR:QFN50P350X350X100-21N
- U2: value BQ25570RGRR -> MAX9934TAUA; device BQ25570RGRR:QFN50P350X350X100-21N -> MAX9934TAUA:21-0036K
- U3: value TSU111ICT -> MAX9934TAUA; device TSU111ICT:SC70-5 -> MAX9934TAUA:21-0036K
- U4: value MAX9934TAUA -> MAX9620; device MAX9934TAUA:21-0036K -> MAX9620:SC70-5
- U5, U6: value TSU111ICT -> MAX9620; device TSU111ICT:SC70-5 -> MAX9620:SC70-5
- moved C23 61.9 mm to (62.5, 5.00), flipped to the top, turned to 180 degrees
- moved R14 61.0 mm to (69.0, 47.0), turned to 270 degrees
- moved R8 56.3 mm to (64.0, 12.0), flipped to the bottom, turned to 180 degrees
- moved J2 55.4 mm to (6.00, 41.0), turned to 90 degrees
- moved R15 55.3 mm to (65.0, 47.0), turned to 90 degrees
- moved U4 53.7 mm to (65.5, 7.00), flipped to the top, turned to 90 degrees
- moved R10 52.3 mm to (31.0, 11.0)
- moved R9 52.3 mm to (27.0, 11.0), turned to 270 degrees
- moved C1 51.6 mm to (19.0, 15.0), flipped to the top
- moved J3 49.5 mm to (41.0, 6.00), turned to 180 degrees
- moved C19 48.6 mm to (55.0, 10.0), flipped to the bottom
- moved SJ15 48.1 mm to (57.0, 3.00), turned to 0 degrees
- moved R19 47.2 mm to (14.0, 55.0)
- moved R5 43.9 mm to (19.0, 11.0), flipped to the top
- moved C18 43.4 mm to (28.0, 44.0), turned to 180 degrees
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Connections:
- removed net N$15 (its old number): R5.1, U3.3, U3.4
- removed net N$19: Q2.3, R10.2, R9.1
- new net N$25: Q2.3, R14.2, R15.1
- new net N$9: R18.1, U4.3, U4.4
- net CMES1: now also C2.1, C4.1, R1.2, U2.2; no longer C11.1, C8.1, R6.2, U4.2
- net CMES2: now also C5.1, U3.2; no longer C1.1, U1.2
- net GND: now also C10.1, C16.2, C17.2, C5.2, C6.2, C7.1, C8.1, C9.1, J5.1, J7.2, J7.S1, J7.S2, R1.1, R13.1, R20.1, R5.1, U1.1, U1.15, U1.17, U1.21, U1.22, U1.23, U1.24, U1.25, U1.9, U2.3, U3.3, U4.2; no longer C10.2, C16.1, C17.1, C5.1, C6.1, C7.2, C8.2, C9.2, J5.2, J5.S1, J5.S2, R12.1, R16.1, R23.1, R3.1, U1.3, U2.1, U2.15, U2.17, U2.21, U2.22, U2.23, U2.24, U2.25, U2.9, U3.2, U4.3
- net LBOOST: now also U1.20; no longer U2.20
- net LBUCK: now also U1.16; no longer U2.16
- net N$1: now also C18.1, SJ3.1, U2.8; no longer C22.1, SJ9.1, U4.8
- net N$10: now also C21.1, U3.7; no longer C20.1, U1.7
- net N$11: now also C19.1, U3.8; no longer C18.1, U1.8
- net N$12: now also R19.2; no longer C24.1, R20.2
- net N$13: now also R18.2, SJ17.3; no longer C25.1, R21.2, SJ19.3
- net N$14: now also SJ15.2, U4.1; no longer SJ12.2, U6.1
- net N$16: now also R21.2, SJ19.3; no longer C10.1, R5.2, SJ3.3
- net N$17: now also R16.2, R17.2, SJ14.1, U6.1; no longer R1.2, R3.2, SJ1.1, U3.1
- net N$18: now also R16.1, SJ14.3; no longer R1.1, SJ1.3
- net N$2: now also R20.2, R22.1; no longer R12.2, R13.1
- net N$20: now also R15.2; no longer R9.2
- net N$21: now also SJ13.3; no longer SJ8.3
- net N$23: now also R14.1; no longer R10.1
- net N$3: now also R22.2, R23.1; no longer R13.2, R14.1
- net N$4: now also R7.2, U2.6; no longer R11.2, U4.6
- net N$5: now also R19.1; no longer R20.1
- net N$6: now also C20.1, SJ5.1, U2.7; no longer C23.1, SJ10.1, U4.7
- net N$7: now also R8.2, U3.6; no longer R7.2, U1.6
- net N$8: now also SJ16.2; no longer SJ11.2
- net NEN: now also U1.5; no longer U2.5
- net OK_HYST: now also R10.2, R9.1, U1.10; no longer R18.1, R19.2, U2.10
- net OK_PROG: now also R10.1, R6.2, U1.11; no longer R17.2, R19.1, U2.11
- net RSN2: now also J3.2, R3.P$3, R3.P$4, SJ1.2, SJ13.1, SJ15.1, SJ17.1; no longer J2.2, R4.P$3, R4.P$4, SJ12.1, SJ19.1, SJ2.2, SJ8.1
- net RSN2_BUF: now also SJ17.2; no longer SJ19.2
- net RSP1: now also J2.2, R11.P$3, R11.P$4, SJ16.1, SJ2.2; no longer J3.2, R8.P$3, R8.P$4, SJ10.2, SJ11.1
- net SW: now also J7.1; no longer J5.1
- net VBAT: now also C22.1, SJ14.2, SJ19.1, U1.18; no longer C21.1, SJ1.2, SJ3.1, U2.18
- net VBAT_BUF: now also SJ19.2; no longer SJ3.2
- net VBAT_OK: now also U1.13; no longer U2.13
- net VBAT_OV: now also R4.1, R5.2, U1.7; no longer R15.1, R16.2, U2.7
- net VCC_SW: now also J5.2, SJ10.1, SJ11.1, SJ12.1, SJ13.2, SJ8.1, SJ9.1; no longer SJ13.1, SJ14.1, SJ15.1, SJ16.1, SJ17.1, SJ8.2
- net VCC_SW1: now also C7.2, C8.2, R7.1, SJ8.2, U2.1; no longer C16.2, C17.2, R11.1, SJ13.2, U4.1
- net VCC_SW2: now also C10.2, C9.2, R8.1, SJ9.2, U3.1; no longer C5.2, C6.2, R7.1, SJ14.2, U1.1
- net VCC_SW3: now also C24.1, SJ10.2; no longer SJ15.2
- net VCC_SW4: now also C23.1, SJ11.2, U4.5; no longer SJ16.2, U6.5
- net VCC_SW5: now also C25.1, SJ12.2, U6.5; no longer SJ17.2, U3.5
- net VIN_DC: now also C14.1, C16.1, C17.1, R11.P$1, R11.P$2, R23.2, SJ2.1, SJ3.2, U1.2; no longer C13.1, C15.1, C19.1, R14.2, R8.P$1, R8.P$2, SJ5.1, SJ9.2, U2.2
- net VOC_SAMP: now also U1.3; no longer U2.3
- net VOUT: now also C11.1, C6.1, R3.P$1, R3.P$2, SJ1.1, U1.14; no longer C4.1, C7.1, R4.P$1, R4.P$2, SJ2.1, U2.14
- net VOUT_EN: now also U1.6; no longer U2.6
- net VOUT_SET: now also R12.1, R13.2, U1.12; no longer R22.1, R23.2, U2.12
- net VRDIV: now also R12.2, R4.2, R9.2, U1.8; no longer R15.2, R18.2, R22.2, U2.8
- net VREF_SAMP: now also C1.1, U1.4; no longer C2.1, U2.4
- net VSTOR: now also C13.1, C15.1, U1.19; no longer C14.1, C9.1, U2.19
Routing:
- net VCC_SW: track 30.8 -> 53.4 mm, vias 0 -> 1
- net N$25: track 0.00 -> 8.26 mm
- net N$19: track 8.26 -> 0.00 mm
- net SW: track 10.9 -> 17.1 mm
- net N$13: track 18.3 -> 13.2 mm
- net N$15 (its old number): track 4.66 -> 0.00 mm
- net N$9: track 0.00 -> 4.25 mm
- net VCC_SW4: track 63.4 -> 67.6 mm
- net VCC_SW5: track 13.1 -> 16.4 mm
- net VCC_SW3: track 44.3 -> 47.0 mm
- net N$14: track 14.6 -> 16.0 mm
- net N$5: track 7.03 -> 7.99 mm
- net N$15: track 4.03 -> 4.66 mm
- net GND: vias 67 -> 71
Other:
- board text added: "Energy Harvesting Monitor V1.2"
- board text added: "OUT_SW"
- board text removed: "Energy Harvesting Monitor V1.0"

Commit message: Added resistor to base of high side switch
Parts:
- added R24: DNP, rcl:R0603
Connections:
- new net N$19: Q2.2, R24.1
- net SW: now also R24.2; no longer Q2.2
Routing:
- net SW: track 17.1 -> 10.2 mm
- net N$19: track 0.00 -> 5.24 mm
Changed lines of the file:
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@@
 <attribute name="VALUE" x="67.49363125" y="40.00425" size="0.81395" layer="27" rot="R270"/>
+</element>
+<element name="R24" library="rcl" library_urn="urn:adsk.eagle:library:334" package="R0603" package3d_urn="urn:adsk.eagle:package:23555/2" value="DNP" x="64" y="34" smashed="yes" rot="R270">
+<attribute name="NAME" x="62.865" y="32.365" size="1.27" layer="25" rot="R90"/>
+<attribute name="SPICEPREFIX" value="R" x="64" y="34" size="1.778" layer="27" rot="R270" display="off"/>
+<attribute name="VALUE" x="62.095" y="34.635" size="1.27" layer="27" rot="R270"/>
 </element>
 </elements>
@@
 <signal name="SW">
 <contactref element="J7" pad="1"/>
-<contactref element="Q2" pad="2"/>
-<wire x1="64" y1="29" x2="66.5" y2="26.5" width="0.508" layer="1"/>
-<wire x1="64" y1="40.095" x2="64" y2="29" width="0.508" layer="1"/>
-<wire x1="66.5" y1="26.5" x2="69" y2="26.5" width="0.508" layer="1"/>
+<contactref element="R24" pad="2"/>
+<wire x1="69" y1="26.5" x2="66.5" y2="26.5" width="0.508" layer="1"/>
+<wire x1="66.5" y1="26.5" x2="64" y2="29" width="0.508" layer="1"/>
+<wire x1="64" y1="29" x2="64" y2="33.15" width="0.508" layer="1"/>
 </signal>
 <signal name="N$21">
@@
 <wire x1="65.27" y1="45.88" x2="65" y2="46.15" width="0.6096" layer="1"/>
 </signal>
+<signal name="N$19">
+<contactref element="R24" pad="1"/>
+<contactref element="Q2" pad="2"/>
+<wire x1="64" y1="34.85" x2="64" y2="40.095" width="0.508" layer="1"/>
+</signal>
 </signals>

Commit message: Updated to V1.4
Parts:
- added R25: 0R, rcl:R0603
- added R26: 7.87M, rcl:R0603
- added TP27: TPB1,27, testpad:B1,27
- R1: value (none) -> 10.7k
- R10, R12: value (none) -> 7.15M
- R11: value (none) -> 0.05R
- R13: value (none) -> 5.76M
- R14, R7, R8: value DNP -> 10k
- R15: value DNP -> 2.2k
- R16: value DNP -> 18k
- R17, R18, R19, R20: value DNP -> 10M
- R2: value (none) -> 9.31k
- R21: value DNP -> 5.23M
- R22, R23, R24: value DNP -> 0R
- R3: value (none) -> 0.1R
- R4: value (none) -> 7.32M
- R5: value (none) -> 5.62M
- R6: value (none) -> 5.11M
- R9: value (none) -> 866k
- SJ13: device jumper:SJ_2 -> jumper:SJ
- SJ15, SJ8: device jumper:SJ -> jumper:SJ_2
- TP11, TP16: value TPPAD1-13Y -> TPPAD1-13; device testpad:P1-13Y -> testpad:P1-13
- TP19: value TPPAD1-13Y -> TPB1,27; device testpad:P1-13Y -> testpad:B1,27
- moved SJ16 60.5 mm to (57.0, 3.00), turned to 0 degrees
- moved R18 59.3 mm to (25.0, 55.5), turned to 90 degrees
- moved SJ15 57.3 mm to (25.0, 50.5), turned to 90 degrees
- moved R19 47.0 mm to (55.0, 32.0), flipped to the bottom, turned to 90 degrees
- moved R21 45.9 mm to (12.5, 16.0), flipped to the top
- moved R22 43.9 mm to (51.0, 41.0), flipped to the bottom
- moved R20 40.6 mm to (22.0, 55.5), turned to 270 degrees
- moved U4 32.5 mm to (53.0, 37.0), flipped to the bottom, turned to 0 degrees
- moved U6 32.5 mm to (65.5, 7.00), flipped to the top, turned to 90 degrees
- moved R23 31.6 mm to (10.5, 55.5), turned to 270 degrees
- moved C23 31.1 mm to (56.5, 35.5), flipped to the bottom
- moved C25 31.1 mm to (62.5, 5.00), flipped to the top
- moved SJ17 29.2 mm to (60.0, 36.0), flipped to the bottom, turned to 90 degrees
- moved SJ19 29.2 mm to (57.0, 7.00), flipped to the top, turned to 0 degrees
- moved R24 24.5 mm to (62.5, 9.50), turned to 180 degrees
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Connections:
- new net N$26: R18.1, SJ15.3, TP27.TP
- net GND: now also R19.1, R21.1; no longer R17.1
- net N$12: now also R23.2; no longer R19.2
- net N$13: now also R24.2, SJ19.3; no longer R18.2, SJ17.3
- net N$14: now also SJ16.2, U6.1; no longer SJ15.2, U4.1
- net N$15: now also R22.1, U4.3, U4.4; no longer R21.1, U6.3, U6.4
- net N$16: now also R22.2, SJ17.3; no longer R21.2, SJ19.3
- net N$17: now also R19.2, U4.1; no longer R16.2, U6.1
- net N$18: now also R17.1; no longer R16.1
- net N$19: now also R16.1; no longer R24.1
- net N$2: now also R21.2, R25.1; no longer R20.2, R22.1
- net N$21: now also SJ8.3; no longer SJ13.3
- net N$3: now also R25.2, R26.1; no longer R22.2, R23.1
- net N$5: now also R23.1; no longer R19.1
- net N$8: now also R18.2, R20.2, SJ15.1; no longer SJ16.2
- net N$9: now also R24.1, U6.3, U6.4; no longer R18.1, U4.3, U4.4
- net RSN2: now also SJ16.1, SJ19.1, SJ8.1; no longer SJ13.1, SJ15.1, SJ17.1
- net RSN2_BUF: now also SJ19.2; no longer SJ17.2
- net RSP1: now also SJ15.2; no longer SJ16.1
- net SW: now also R16.2; no longer R24.2
- net VBAT: now also SJ17.1; no longer SJ19.1
- net VBAT_BUF: now also SJ17.2; no longer SJ19.2
- net VCC_SW: now also SJ13.1, SJ8.2; no longer SJ13.2, SJ8.1
- net VCC_SW1: now also SJ9.2; no longer SJ8.2
- net VCC_SW2: now also SJ10.2; no longer SJ9.2
- net VCC_SW3: now also SJ11.2; no longer SJ10.2
- net VCC_SW4: now also C25.1, SJ12.2, U6.5; no longer C23.1, SJ11.2, U4.5
- net VCC_SW5: now also C23.1, SJ13.2, U4.5; no longer C25.1, SJ12.2, U6.5
- net VIN_DC: now also R26.2; no longer R23.2
Routing:
- net RSP1: track 7.64 -> 20.0 mm, vias 2 -> 4
- net VCC_SW3: track 47.0 -> 56.1 mm
- net N$26: track 0.00 -> 6.10 mm
- net N$5: track 7.99 -> 12.6 mm
- net N$12: track 12.3 -> 7.76 mm
- net N$8: track 14.9 -> 19.0 mm, vias 2 -> 0
- net RSP1_BUF: track 31.3 -> 34.2 mm
- net GND: vias 71 -> 69
Other:
- board text added: "Energy Harvesting Monitor V1.4"
- board text removed: "Energy Harvesting Monitor V1.2"

Commit message: First commit to develop branch
Parts:
- removed C25: 0.1uF, rcl:C0603
- removed Q1: BC557B, transistor-pnp:TO92-EBC
- removed Q2: BC547B, transistor-npn:TO92
- removed R25: 0R, rcl:R0603
- removed R26: 7.87M, rcl:R0603
- removed SJ16: (no value), jumper:SJ
- removed SJ17, SJ18, SJ19: (no value), jumper:SJ_2
- removed TP27: TPB1,27, testpad:B1,27
- added F1: 1206L012THR, 1206L012THR:R1206
- added U7: ADS7041IRUGR, ADS7041IRUG:QFN50P150X150X40-8N
- C12: value 0.1uF -> 4.7uF
- C13, C7: value 4.7uF -> DNP
- C14: value 0.1uF -> DNP
- C16: value 4.7uF -> 0.1uF
- C17, C19: value DNP -> 0.1uF
- C18: value DNP -> 100uF; device rcl:C0805 -> rcl:C1210
- C2: value DNP -> 4.7uF; device rcl:C1210 -> rcl:C0805
- C22: value DNP -> 1.5nF; device rcl:C1812 -> rcl:C0603
- C23, C24: value 0.1uF -> 1uF; device rcl:C0603 -> rcl:C0805
- C3: value DNP -> 0.1uF; device rcl:C1210 -> rcl:C0805
- C4: value 0.01uF -> 4.7uF
- C5: value 0.01uF -> 0.1uF
- J6: value S6B-PH-SM4-TB(LF)(SN) -> SM02B-SRSS-TB(LF)(SN); device S6B-PH-SM4-TB_LF__SN_:JST_S6B-PH-SM4-TB(LF)(SN) -> SM02B-SRSS-TB(LF)(SN):SM02B-SRSS-TB
- J7: value S2B-PH-SM4-TB(LF)(SN) -> SM06B-SRSS-TB(LF)(SN); device S2B-PH-SM4-TB_LF__SN_:JST_S2B-PH-SM4-TB(LF)(SN) -> SM06B-SRSS-TB(LF)(SN):SM06B-SRSS-B
- R14: value 10k -> 50R
- R15: value 2.2k -> 50R
- R16: value 18k -> 10M
- R20: value 10M -> 5.23M
- R21: value 5.23M -> 0R
- R22: value 0R -> 7.87M
- R23: value 0R -> 50R
- R24: value 0R -> 200R
- R6: value 5.11M -> 10k
- R8: value 10k -> 5.11M
- SJ11, SJ12, SJ13, SJ3: device jumper:SJ -> jumper:SJ_2
- SJ8: device jumper:SJ_2 -> jumper:SJ
- TP1, TP12, TP24, TP4, TP6, TP7, TP8: value TPPAD1-13Y -> TPPAD1-13; device testpad:P1-13Y -> testpad:P1-13
- TP10, TP18, TP9: value TPPAD1-13 -> TPB1,27; device testpad:P1-13 -> testpad:B1,27
- TP17, TP20, TP21, TP22, TP3: value TPPAD1-13Y -> TPB1,27; device testpad:P1-13Y -> testpad:B1,27
- TP19, TP23: value TPB1,27 -> TPPAD1-13; device testpad:B1,27 -> testpad:P1-13
- U1: value BQ25570RGRR -> MAX9934TAUA; device BQ25570RGRR:QFN50P350X350X100-21N -> MAX9934TAUA:21-0036K
- U3: value MAX9934TAUA -> BQ25570RGRR; device MAX9934TAUA:21-0036K -> BQ25570RGRR:QFN50P350X350X100-21N
- U4: value MAX9620 -> MAX4715; device MAX9620:SC70-5 -> MAX4715:SC70-5L
- U5: value MAX9620 -> OPA314IDCKR; device MAX9620:SC70-5 -> OPA314IDCK:SC70-5L
- U6: value MAX9620 -> DG2034EDQ-T1-GE3; device MAX9620:SC70-5 -> DG2034EDQ-T1-GE3:MSOP10
- moved R23 62.5 mm to (71.5, 42.0), turned to 90 degrees
- moved C24 58.8 mm to (72.0, 49.5), turned to 0 degrees
- moved J6 55.9 mm to (80.0, 13.0), turned to 90 degrees
- moved C3 54.1 mm to (24.0, 51.5), turned to 270 degrees
- moved SJ5 51.6 mm to (65.0, 20.0), flipped to the top, turned to 90 degrees
- moved SJ9 49.5 mm to (56.0, 7.50)
- moved C22 49.2 mm to (67.5, 51.0), flipped to the top
- moved U5 46.9 mm to (64.5, 46.0), turned to 180 degrees
- moved SJ3 46.0 mm to (56.5, 12.5), flipped to the top
- moved C10 42.5 mm to (20.5, 24.0), flipped to the top
- moved C17 42.2 mm to (50.5, 28.5), flipped to the bottom, turned to 90 degrees
- moved R22 42.1 mm to (12.5, 24.0), flipped to the top
- moved C20 42.1 mm to (66.0, 42.0), flipped to the top, turned to 0 degrees
- moved U6 41.7 mm to (49.5, 45.5), turned to 0 degrees
- moved R24 41.5 mm to (64.5, 51.0), turned to 270 degrees
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Connections:
- removed net N$1: C18.1, SJ3.1, U2.8
- removed net N$11: C19.1, SJ4.1, U3.8
- removed net N$14: SJ16.2, TP18.TP, U6.1
- removed net N$15: R22.1, U4.3, U4.4
- removed net N$16: R22.2, SJ17.3, TP22.TP
- removed net N$17: R17.2, R19.2, SJ14.1, TP21.TP, U4.1
- removed net N$18: R17.1, SJ14.3, TP20.TP
- removed net N$19: Q2.2, R16.1
- removed net N$20: Q1.B, R15.2
- removed net N$21: Q1.C, SJ8.3
- removed net N$23: Q1.E, R14.1, SJ7.2
- removed net N$25: Q2.3, R14.2, R15.1
- removed net N$26: R18.1, SJ15.3, TP27.TP
- removed net N$7 (its old number): R8.2, U3.6
- removed net RSN2_BUF: J6.4, SJ19.2
- removed net RSP1_BUF: J6.3, SJ18.2
- removed net VBAT_BUF: J6.5, SJ17.2
- new net !CS!: R14.1, TP20.TP, U7.1
- new net A0: J7.1, U6.1
- new net A1: J7.2, U6.10
- new net BUF_IN: SJ10.1, SJ11.1, SJ12.3, SJ13.1, SJ14.1, SJ15.3, U6.8
- new net BUF_OUT: R24.2, SJ13.2
- new net N$27: SJ13.3, U5.3, U5.4
- new net N$4: R6.2, U1.6
- new net RSP1_DIV: R16.1, R17.2, SJ11.2, TP16.TP
- new net S1: SJ11.3, U6.2
- new net S2: SJ12.1, U6.9
- new net S3: SJ14.3, U6.4
- new net S4: SJ15.1, U6.7
- new net SCLK: R15.1, TP22.TP, U7.3
- new net SDO: J7.4, R23.1, TP21.TP
- new net V+: C19.1, SJ9.1, U4.2, U4.5
- new net VBAT_DIV: R18.1, R19.2, SJ12.2, TP19.TP
- net CMES1: now also SJ15.2, U1.2; no longer C2.1, C4.1, J6.1, U2.2
- net CMES2: now also SJ14.2, U2.2; no longer C3.1, C5.1, J6.2, U3.2
- net GND: now also C10.2, C2.1, C22.1, C23.1, C3.1, C4.1, C5.1, C7.2, C8.2, C9.2, J6.2, J6.3, J6.4, J7.6, J7.7, J7.8, R17.1, R8.1, U1.3, U3.1, U3.15, U3.17, U3.21, U3.22, U3.23, U3.24, U3.25, U3.9, U4.3, U6.3, U7.5, U7.8; no longer C10.1, C2.2, C22.2, C23.2, C25.2, C3.2, C4.2, C5.2, C7.1, C8.1, C9.1, J6.6, J6.S1, J6.S2, J7.2, J7.S1, J7.S2, Q2.1, R21.1, R6.1, U1.1, U1.15, U1.17, U1.21, U1.22, U1.23, U1.24, U1.25, U1.9, U3.3, U4.2, U6.2
- net LBOOST: now also U3.20; no longer U1.20
- net LBUCK: now also U3.16; no longer U1.16
- net N$10: now also SJ3.3, U4.1; no longer C21.1, SJ6.1, U3.7
- net N$12: now also J7.5, R15.2; no longer R23.2, SJ18.3, TP16.TP
- net N$13: now also C22.2, R24.1, U7.7; no longer R24.2, SJ19.3
- net N$2: now also R20.2, R21.1; no longer R21.2, R25.1
- net N$3: now also R21.2, R22.1; no longer R25.2, R26.1
- net N$5: now also R23.2, U7.2; no longer R23.1, U5.3, U5.4
- net N$6: now also F1.2, J5.2; no longer C20.1, SJ5.1, U2.7
- net N$8: now also SJ10.2, TP14.TP; no longer R18.2, R20.2, SJ15.1, TP19.TP
- net N$9: now also J7.3, R14.2; no longer R24.1, U6.3, U6.4
- net NEN: now also U3.5; no longer U1.5
- net OK_HYST: now also U3.10; no longer U1.10
- net OK_PROG: now also R8.2, U3.11; no longer R6.2, U1.11
- net RSN2: now also C14.1, SJ3.1, SJ9.2, U2.8; no longer SJ16.1, SJ19.1, SJ4.2, SJ7.1, SJ8.1
- net RSP1: now also C16.1, R16.2, U1.7; no longer SJ15.2, SJ18.1, SJ5.2
- net SW: now also J6.1, U4.4; no longer J7.1, R16.2
- net VBAT: now also C18.1, R18.2, U3.18; no longer C22.1, SJ14.2, SJ17.1, U1.18
- net VBAT_OK: now also U3.13; no longer U1.13
- net VBAT_OV: now also U3.7; no longer U1.7
- net VCC_SW: now also F1.1, SJ3.2, SJ4.1, SJ5.1, SJ6.1, SJ7.1, SJ8.1; no longer J5.2, SJ10.1, SJ11.1, SJ12.1, SJ13.1, SJ8.2, SJ9.1
- net VCC_SW1: now also C2.2, C3.2, R6.1, SJ4.2, U1.1; no longer C7.2, C8.2, R7.1, SJ9.2, U2.1
- net VCC_SW2: now also C4.2, C5.2, R7.1, SJ5.2, U2.1; no longer C10.2, C9.2, R8.1, SJ10.2, U3.1
- net VCC_SW3: now also C21.1, SJ6.2, U6.5, U6.6; no longer C24.1, SJ11.2, U5.5
- net VCC_SW4: now also C20.1, SJ7.2, TP15.TP, U5.5; no longer C25.1, SJ12.2, TP14.TP, U6.5
- net VCC_SW5: now also C23.2, C24.1, SJ8.2, TP18.TP, U7.4, U7.6; no longer C23.1, SJ13.2, TP15.TP, U4.5
- net VIN_DC: now also C10.1, C12.1, C13.1, C15.1, R22.2, U1.8, U3.2; no longer C14.1, C16.1, C17.1, R26.2, SJ3.2, U1.2
- net VOC_SAMP: now also U3.3; no longer U1.3
- net VOUT: now also C17.1, C7.1, U2.7, U3.14; no longer C11.1, SJ6.2, U1.14
- net VOUT_EN: now also U3.6; no longer U1.6
- net VOUT_SET: now also U3.12; no longer U1.12
- net VRDIV: now also U3.8; no longer U1.8
- net VREF_SAMP: now also U3.4; no longer U1.4
- net VSTOR: now also C11.1, C8.1, C9.1, U3.19; no longer C12.1, C13.1, C15.1, U1.19
Routing:
- net RSN2: track 90.8 -> 11.4 mm
- net RSN2_BUF: track 57.1 -> 0.00 mm, vias 6 -> 0
- net VCC_SW5: track 16.4 -> 55.5 mm, vias 2 -> 4
- net VCC_SW2: track 67.8 -> 28.9 mm, vias 6 -> 3
- net A1: track 0.00 -> 37.6 mm, vias 0 -> 2
- net A0: track 0.00 -> 37.2 mm, vias 0 -> 2
- net VBAT_BUF: track 36.9 -> 0.00 mm, vias 3 -> 0
- net VCC_SW4: track 67.6 -> 32.3 mm, vias 7 -> 1
- net BUF_IN: track 0.00 -> 34.2 mm
- net RSP1_BUF: track 34.2 -> 0.00 mm, vias 2 -> 0
- net CMES2: track 61.9 -> 32.3 mm, vias 3 -> 1
- net VBAT: track 153.5 -> 126.0 mm, vias 3 -> 2
- net VCC_SW1: track 43.4 -> 67.9 mm, vias 2 -> 4
- net N$16: track 23.9 -> 0.00 mm, vias 2 -> 0
- net N$17: track 20.3 -> 0.00 mm
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- added copper zone on layer 1, net N$14
- added copper zone on layer 16, net RSN2
- added copper zone on layer 16, net RSP1
- added copper zone on layer 1, net VCC_SW3
- added copper zone on layer 1, net VCC_SW5
- added copper zone on layer 16, net VIN_DC
- added copper zone on layer 16, net VOUT
- removed copper zone on layer 1, net N$24
Other:
- board size 78 x 60 mm -> 85 x 55 mm
- board text added: "!CS!"
- board text added: "A"
- board text added: "A0"
- board text added: "A1"
- board text added: "B"
- board text added: "Energy Harvesting Monitor V2.0"
- board text added: "OSWF"
- board text added: "SCLK"
- board text added: "SDO"
- board text removed: "CIB"
- board text removed: "COB"
- board text removed: "Energy Harvesting Monitor V1.4"
- board text removed: "OUT_SW"
- board text removed: "VBB"
- board text removed: "VIB"
- board text removed: "VOB"
