File: Project/EHM.brd (EAGLE design)
At the start: 85 x 55 mm, 108 parts, among them J1 282834-2, J2 282834-2, J3 282834-2, J4 282834-2, J5 282834-2, J6 SM02B-SRSS-TB(LF)(SN), J7 SM06B-SRSS-TB(LF)(SN), U1 MAX9934TAUA, U2 MAX9934TAUA, U3 BQ25570RGRR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

Commit message: Added OSHW logo
Parts:
- added U$1: (no value), OSHW:OSHW_8MM
Changed lines of the file:
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@@
 <attribute name="VALUE" x="50.46" y="49.73" size="1.27" layer="28" rot="MR90"/>
 </element>
+<element name="U$1" library="OSHW" package="OSHW_8MM" value="" x="15.5" y="30" smashed="yes" rot="MR90"/>
 </elements>
 <signals>
@@
 </drawing>
 <compatibility>
+<note version="6.3" minversion="6.2.2" severity="warning">
+Since Version 6.2.2 text objects can contain more than one line,
+which will not be processed correctly with this version.
+</note>
 <note version="8.2" severity="warning">
 Since Version 8.2, EAGLE supports online libraries. The ids
