File: Project/EHM.sch (EAGLE design)
At the start: 116 parts, among them J1 282834-2, J2 282834-2, J3 282834-2, J4 282834-2, J5 282834-2, J6 S6B-PH-SM4-TB(LF)(SN), J7 S2B-PH-SM4-TB(LF)(SN), Q1 BC557B, Q2 BC547B, U1 BQ25570RGRR, U2 MAX9934TAUA, U3 MAX9934TAUA, U4 MAX9620, U5 MAX9620, U6 MAX9620

Commit message: First commit to develop branch
Parts:
- removed C25: 0.1uF, rcl:C-EUC0603
- removed Q1: BC557B, transistor-pnp:BC557B
- removed Q2: BC547B, transistor-npn:BC547B
- removed R25: 0R, rcl:R-EU_R0603
- removed R26: 7.87M, rcl:R-EU_R0603
- removed SJ16: (no value), jumper:SJ
- removed SJ17, SJ18, SJ19: (no value), jumper:SJ2W
- removed TP27: TPB1,27, testpad:TPB1,27
- added F1: 1206L012THR, 1206L012THR:1206L012THR
- added U7: ADS7041IRUGR, ADS7041IRUG:ADS7041IRUGR
- C12: value 0.1uF -> 4.7uF
- C13, C7: value 4.7uF -> DNP
- C14: value 0.1uF -> DNP
- C16: value 4.7uF -> 0.1uF
- C17, C19: value DNP -> 0.1uF
- C18: value DNP -> 100uF; device rcl:C-EUC0805 -> rcl:C-EUC1210
- C2: value DNP -> 4.7uF; device rcl:C-EUC1210 -> rcl:C-EUC0805
- C22: value DNP -> 1.5nF; device rcl:C-EUC1812 -> rcl:C-EUC0603
- C23, C24: value 0.1uF -> 1uF; device rcl:C-EUC0603 -> rcl:C-EUC0805
- C3: value DNP -> 0.1uF; device rcl:C-EUC1210 -> rcl:C-EUC0805
- C4: value 0.01uF -> 4.7uF
- C5: value 0.01uF -> 0.1uF
- J6: value S6B-PH-SM4-TB(LF)(SN) -> SM02B-SRSS-TB(LF)(SN); device S6B-PH-SM4-TB_LF__SN_:S6B-PH-SM4-TB(LF)(SN) -> SM02B-SRSS-TB(LF)(SN):SM02B-SRSS-TB(LF)(SN)
- J7: value S2B-PH-SM4-TB(LF)(SN) -> SM06B-SRSS-TB(LF)(SN); device S2B-PH-SM4-TB_LF__SN_:S2B-PH-SM4-TB(LF)(SN) -> SM06B-SRSS-TB(LF)(SN):SM06B-SRSS-TB(LF)(SN)
- R14: value 10k -> 50R
- R15: value 2.2k -> 50R
- R16: value 18k -> 10M
- R20: value 10M -> 5.23M
- R21: value 5.23M -> 0R
- R22: value 0R -> 7.87M
- R23: value 0R -> 50R
- R24: value 0R -> 200R
- R6: value 5.11M -> 10k
- R8: value 10k -> 5.11M
- SJ11, SJ12, SJ13, SJ3: device jumper:SJ -> jumper:SJ2W
- SJ8: device jumper:SJ2W -> jumper:SJ
- TP1, TP12, TP24, TP4, TP6, TP7, TP8: value TPPAD1-13Y -> TPPAD1-13; device testpad:TPPAD1-13Y -> testpad:TPPAD1-13
- TP10, TP18, TP9: value TPPAD1-13 -> TPB1,27; device testpad:TPPAD1-13 -> testpad:TPB1,27
- TP17, TP20, TP21, TP22, TP3: value TPPAD1-13Y -> TPB1,27; device testpad:TPPAD1-13Y -> testpad:TPB1,27
- TP19, TP23: value TPB1,27 -> TPPAD1-13; device testpad:TPB1,27 -> testpad:TPPAD1-13
- U1: value BQ25570RGRR -> MAX9934TAUA; device BQ25570RGRR:BQ25570RGRR -> MAX9934TAUA:MAX9934TAUA
- U3: value MAX9934TAUA -> BQ25570RGRR; device MAX9934TAUA:MAX9934TAUA -> BQ25570RGRR:BQ25570RGRR
- U4: value MAX9620 -> MAX4715; device MAX9620:MAX9620 -> MAX4715:MAX4715
- U5: value MAX9620 -> OPA314IDCKR; device MAX9620:MAX9620 -> OPA314IDCK:OPA314IDCKR
- U6: value MAX9620 -> DG2034EDQ-T1-GE3; device MAX9620:MAX9620 -> DG2034EDQ-T1-GE3:DG2034EDQ-T1-GE3
Connections:
- removed net N$1: C18.1, SJ3.1, U2.RSN
- removed net N$11: C19.1, SJ4.1, U3.RSN
- removed net N$14: SJ16.2, TP18.TP, U6.IN+
- removed net N$15: R22.1, U4.IN-, U4.OUT
- removed net N$16: R22.2, SJ17.3, TP22.TP
- removed net N$17: R17.2, R19.2, SJ14.1, TP21.TP, U4.IN+
- removed net N$18: R17.1, SJ14.3, TP20.TP
- removed net N$19: Q2.B, R16.1
- removed net N$20: Q1.B, R15.2
- removed net N$21: Q1.C, SJ8.3
- removed net N$23: Q1.E, R14.1, SJ7.2
- removed net N$25: Q2.C, R14.2, R15.1
- removed net N$26: R18.1, SJ15.3, TP27.TP
- removed net N$7 (its old number): R8.2, U3.CS
- removed net RSN2_BUF: J6.4, SJ19.2
- removed net RSP1_BUF: J6.3, SJ18.2
- removed net VBAT_BUF: J6.5, SJ17.2
- new net !CS!: R14.1, TP20.TP, U7.!CS!
- new net A0: J7.1, U6.A0
- new net A1: J7.2, U6.A1
- new net BUF_IN: SJ10.1, SJ11.1, SJ12.3, SJ13.1, SJ14.1, SJ15.3, U6.COM
- new net BUF_OUT: R24.2, SJ13.2
- new net N$27: SJ13.3, U5.IN-, U5.OUT
- new net N$4: R6.2, U1.CS
- new net RSP1_DIV: R16.1, R17.2, SJ11.2, TP16.TP
- new net S1: SJ11.3, U6.S1
- new net S2: SJ12.1, U6.S2
- new net S3: SJ14.3, U6.S3
- new net S4: SJ15.1, U6.S4
- new net SCLK: R15.1, TP22.TP, U7.SCLK
- new net SDO: J7.4, R23.1, TP21.TP
- new net V+: C19.1, SJ9.1, U4.NO, U4.V+
- new net VBAT_DIV: R18.1, R19.2, SJ12.2, TP19.TP
- net CMES1: now also SJ15.2, U1.OUT; no longer C2.1, C4.1, J6.1, U2.OUT
- net CMES2: now also SJ14.2, U2.OUT; no longer C3.1, C5.1, J6.2, U3.OUT
- net GND: now also C10.2, C2.1, C22.1, C23.1, C3.1, C4.1, C5.1, C7.2, C8.2, C9.2, J6.2, J7.6, R17.1, R8.1, U1.GROUND, U3.EP@1, U3.EP@2, U3.EP@3, U3.EP@4, U3.EP@5, U3.NC1, U3.NC2, U3.VSS@1, U3.VSS@2, U4.GND, U6.GND, U7.AINM, U7.GND; no longer C10.1, C2.2, C22.2, C23.2, C25.2, C3.2, C4.2, C5.2, C7.1, C8.1, C9.1, J6.6, J7.2, Q2.E, R21.1, R6.1, U1.EP@1, U1.EP@2, U1.EP@3, U1.EP@4, U1.EP@5, U1.NC1, U1.NC2, U1.VSS@1, U1.VSS@2, U3.GROUND, U4.VCC-, U6.VCC-
- net LBOOST: now also U3.LBOOST; no longer U1.LBOOST
- net LBUCK: now also U3.LBUCK; no longer U1.LBUCK
- net N$10: now also SJ3.3, U4.COM; no longer C21.1, SJ6.1, U3.RSP
- net N$12: now also J7.5, R15.2; no longer R23.2, SJ18.3, TP16.TP
- net N$13: now also C22.2, R24.1, U7.AINP; no longer R24.2, SJ19.3
- net N$2: now also R20.2, R21.1; no longer R21.2, R25.1
- net N$3: now also R21.2, R22.1; no longer R25.2, R26.1
- net N$5: now also R23.2, U7.SDO; no longer R23.1, U5.IN-, U5.OUT
- net N$6: now also F1.2, J5.2; no longer C20.1, SJ5.1, U2.RSP
- net N$8: now also SJ10.2, TP14.TP; no longer R18.2, R20.2, SJ15.1, TP19.TP
- net N$9: now also J7.3, R14.2; no longer R24.1, U6.IN-, U6.OUT
- net NEN: now also U3.!EN; no longer U1.!EN
- net OK_HYST: now also U3.OK_HYST; no longer U1.OK_HYST
- net OK_PROG: now also R8.2, U3.OK_PROG; no longer R6.2, U1.OK_PROG
- net RSN2: now also C14.1, SJ3.1, SJ9.2, U2.RSN; no longer SJ16.1, SJ19.1, SJ4.2, SJ7.1, SJ8.1
- net RSP1: now also C16.1, R16.2, U1.RSP; no longer SJ15.2, SJ18.1, SJ5.2
- net SW: now also J6.1, U4.IN; no longer J7.1, R16.2
- net VBAT: now also C18.1, R18.2, U3.VBAT; no longer C22.1, SJ14.2, SJ17.1, U1.VBAT
- net VBAT_OK: now also U3.VBAT_OK; no longer U1.VBAT_OK
- net VBAT_OV: now also U3.VBAT_OV; no longer U1.VBAT_OV
- net VCC_SW: now also F1.1, SJ3.2, SJ4.1, SJ5.1, SJ6.1, SJ7.1, SJ8.1; no longer J5.2, SJ10.1, SJ11.1, SJ12.1, SJ13.1, SJ8.2, SJ9.1
- net VCC_SW1: now also C2.2, C3.2, R6.1, SJ4.2, U1.VCC; no longer C7.2, C8.2, R7.1, SJ9.2, U2.VCC
- net VCC_SW2: now also C4.2, C5.2, R7.1, SJ5.2, U2.VCC; no longer C10.2, C9.2, R8.1, SJ10.2, U3.VCC
- net VCC_SW3: now also C21.1, SJ6.2, U6.EN, U6.V+; no longer C24.1, SJ11.2, U5.VCC+
- net VCC_SW4: now also C20.1, SJ7.2, TP15.TP, U5.VCC+; no longer C25.1, SJ12.2, TP14.TP, U6.VCC+
- net VCC_SW5: now also C23.2, C24.1, SJ8.2, TP18.TP, U7.AVDD, U7.DVDD; no longer C23.1, SJ13.2, TP15.TP, U4.VCC+
- net VIN_DC: now also C10.1, C12.1, C13.1, C15.1, R22.2, U1.RSN, U3.VIN_DC; no longer C14.1, C16.1, C17.1, R26.2, SJ3.2, U1.VIN_DC
- net VOC_SAMP: now also U3.VOC_SAMP; no longer U1.VOC_SAMP
- net VOUT: now also C17.1, C7.1, U2.RSP, U3.VOUT; no longer C11.1, SJ6.2, U1.VOUT
- net VOUT_EN: now also U3.VOUT_EN; no longer U1.VOUT_EN
- net VOUT_SET: now also U3.VOUT_SET; no longer U1.VOUT_SET
- net VRDIV: now also U3.VRDIV; no longer U1.VRDIV
- net VREF_SAMP: now also U3.VREF_SAMP; no longer U1.VREF_SAMP
- net VSTOR: now also C11.1, C8.1, C9.1, U3.VSTOR; no longer C12.1, C13.1, C15.1, U1.VSTOR
Other:
- note added: "Analog to Digital Converter"
- note added: "Multiplexer"
- note added: "Power Supply for CSAs, Buffer, ADC and Multiplexer"
- note added: "Voltage Buffer"
- note removed: "Power Supply for CSAs and Buffers"
- note removed: "Voltage Buffers"
